File: ses-motor-shield/schematics/motor-schematic/_autosave-external_power.kicad_sch (KiCad schematic)
At the start: 21 parts, among them J1 EXTERNAL_MOTOR_POWER, J2 Conn_01x03_Female, Q2 TIP3055, U1 LM317_SOT-223, U4 AMS1117-5.0, U6 AMS1117-3.3

Commit message: finished board
Parts:
- gave numbers to parts that had none: 1
Changed lines of the file:
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@@
   (symbol (lib_id "Diode:1N4007") (at 96.52 41.91 180) (unit 1)
     (in_bom yes) (on_board yes) (fields_autoplaced)
-    (property "Reference" "D?" (id 0) (at 96.52 35.56 0))
+    (property "Reference" "D2" (id 0) (at 96.52 35.56 0))
     (property "Value" "1N4007" (id 1) (at 96.52 38.1 0))
     (property "Footprint" "Diode_THT:D_DO-41_SOD81_P10.16mm_Horizontal" (id 2) (at 96.52 37.465 0)
