File: ses-motor-shield/schematics/motor-schematic/connectors.kicad_sch (KiCad schematic)
At the start: 9 parts, among them J10 MOTOR_D_OUT, J11 STEPPER_TERMINAL, J3 Conn_01x20_Female, J4 Conn_01x20_Female, J5 SERVO1, J6 SERVO2, J7 MOTOR_A_OUT, J8 MOTOR_B_OUT, J9 MOTOR_C_OUT

Commit message: finished board
Parts:
- removed J10: MOTOR_D_OUT, TerminalBlock_Phoenix:TerminalBlock_Phoenix_MKDS-1,5-2_1x02_P5.00mm_Horizontal, symbol Connector:Screw_Terminal_01x02
- removed J9: MOTOR_C_OUT, TerminalBlock_Phoenix:TerminalBlock_Phoenix_MKDS-1,5-2_1x02_P5.00mm_Horizontal, symbol Connector:Screw_Terminal_01x02
Connections:
- net OUT2: now also J11.3 (Pin_3); no longer J11.4 (Pin_4)
- net OUT3: now also J11.4 (Pin_4); no longer J11.3 (Pin_3)
Other:
- moved on the sheet: J11
Changed lines of the file:
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@@
     (effects (font (size 1.27 1.27)) (justify left bottom))
   )
-  (text "SESBOARD INTERFACE" (at 76.2 54.61 0)
+  (text "SESBOARD INTERFACE" (at 69.85 57.15 0)
     (effects (font (size 1.27 1.27) bold) (justify left bottom))
   )
@@
     )
   )
-  (global_label "MOTOR_D_OUT-" (shape input) (at 163.83 135.89 180) (fields_autoplaced)
-    (effects (font (size 1.27 1.27) bold) (justify right))
-    (property "Intersheet References" "${INTERSHEET_REFS}" (id 0) (at 146.4703 136.017 0)
-      (effects (font (size 1.27 1.27) bold) (justify right) hide)
-    )
-  )
   (global_label "ENA" (shape input) (at 62.23 88.9 180) (fields_autoplaced)
     (effects (font (size 1.27 1.27) bold) (justify right))
@@
     )
   )
-  (global_label "MOTOR_D_OUT+" (shape input) (at 163.83 133.35 180) (fields_autoplaced)
-    (effects (font (size 1.27 1.27) bold) (justify right))
-    (property "Intersheet References" "${INTERSHEET_REFS}" (id 0) (at 146.4703 133.477 0)
-      (effects (font (size 1.27 1.27) bold) (justify right) hide)
-    )
-  )
   (global_label "STEPPER_IN4" (shape input) (at 62.23 93.98 180) (fields_autoplaced)
     (effects (font (size 1.27 1.27) bold) (justify right))
@@
     )
   )
-  (global_label "OUT4" (shape input) (at 163.83 146.05 0) (fields_autoplaced)
-    (effects (font (size 1.27 1.27) bold) (justify left))
-    (property "Intersheet References" "${INTERSHEET_REFS}" (id 0) (at 171.2716 145.923 0)
+  (global_label "OUT4" (shape input) (at 163.83 118.11 0) (fields_autoplaced)
+    (effects (font (size 1.27 1.27) bold) (justify left))
+    (property "Intersheet References" "${INTERSHEET_REFS}" (id 0) (at 171.2716 117.983 0)
       (effects (font (size 1.27 1.27) bold) (justify left) hide)
     )
@@
     )
   )
-  (global_label "OUT1" (shape input) (at 163.83 153.67 0) (fields_autoplaced)
-    (effects (font (size 1.27 1.27) bold) (justify left))
-    (property "Intersheet References" "${INTERSHEET_REFS}" (id 0) (at 171.2716 153.543 0)
+  (global_label "OUT1" (shape input) (at 163.83 125.73 0) (fields_autoplaced)
+    (effects (font (size 1.27 1.27) bold) (justify left))
+    (property "Intersheet References" "${INTERSHEET_REFS}" (id 0) (at 171.2716 125.603 0)
       (effects (font (size 1.27 1.27) bold) (justify left) hide)
     )
@@
     )
   )
-  (global_label "MOTOR_C_OUT-" (shape input) (at 163.83 119.38 180) (fields_autoplaced)
-    (effects (font (size 1.27 1.27) bold) (justify right))
-    (property "Intersheet References" "${INTERSHEET_REFS}" (id 0) (at 146.4703 119.507 0)
-      (effects (font (size 1.27 1.27) bold) (justify right) hide)
-    )
-  )
   (global_label "MOTOR_B_OUT-" (shape input) (at 163.83 106.68 180) (fields_autoplaced)
     (effects (font (size 1.27 1.27) bold) (justify right))
@@
     )
   )
-  (global_label "12V" (shape input) (at 163.83 156.21 0) (fields_autoplaced)
-    (effects (font (size 1.27 1.27) bold) (justify left))
-    (property "Intersheet References" "${INTERSHEET_REFS}" (id 0) (at 169.9411 156.083 0)
+  (global_label "12V" (shape input) (at 163.83 128.27 0) (fields_autoplaced)
+    (effects (font (size 1.27 1.27) bold) (justify left))
+    (property "Intersheet References" "${INTERSHEET_REFS}" (id 0) (at 169.9411 128.143 0)
       (effects (font (size 1.27 1.27) bold) (justify left) hide)
     )
@@
     )
   )
-  (global_label "OUT3" (shape input) (at 163.83 151.13 0) (fields_autoplaced)
-    (effects (font (size 1.27 1.27) bold) (justify left))
-    (property "Intersheet References" "${INTERSHEET_REFS}" (id 0) (at 171.2716 151.003 0)
-      (effects (font (size 1.27 1.27) bold) (justify left) hide)
-    )
-  )
-  (global_label "OUT2" (shape input) (at 163.83 148.59 0) (fields_autoplaced)
-    (effects (font (size 1.27 1.27) bold) (justify left))
-    (property "Intersheet References" "${INTERSHEET_REFS}" (id 0) (at 171.2716 148.463 0)
+  (global_label "OUT3" (shape input) (at 163.83 120.65 0) (fields_autoplaced)
+    (effects (font (size 1.27 1.27) bold) (justify left))
+    (property "Intersheet References" "${INTERSHEET_REFS}" (id 0) (at 171.2716 120.523 0)
+      (effects (font (size 1.27 1.27) bold) (justify left) hide)
+    )
+  )
+  (global_label "OUT2" (shape input) (at 163.83 123.19 0) (fields_autoplaced)
+    (effects (font (size 1.27 1.27) bold) (justify left))
+    (property "Intersheet References" "${INTERSHEET_REFS}" (id 0) (at 171.2716 123.063 0)
       (effects (font (size 1.27 1.27) bold) (justify left) hide)
     )
@@
     (property "Intersheet References" "${INTERSHEET_REFS}" (id 0) (at 115.3311 93.853 0)
       (effects (font (size 1.27 1.27) bold) (justify left) hide)
-    )
-  )
-  (global_label "MOTOR_C_OUT+" (shape input) (at 163.83 121.92 180) (fields_autoplaced)
-    (effects (font (size 1.27 1.27) bold) (justify right))
-    (property "Intersheet References" "${INTERSHEET_REFS}" (id 0) (at 146.4703 122.047 0)
-      (effects (font (size 1.27 1.27) bold) (justify right) hide)
     )
   )
@@
     (pin "9")
   )
-  (symbol (lib_id "Connector:Screw_Terminal_01x02") (at 168.91 119.38 0) (unit 1)
-    (in_bom yes) (on_board yes) (fields_autoplaced)
-    (property "Reference" "J9" (id 0) (at 171.45 119.3799 0)
-      (effects (font (size 1.27 1.27)) (justify left))
-    )
-    (property "Value" "MOTOR_C_OUT" (id 1) (at 171.45 121.9199 0)
-      (effects (font (size 1.27 1.27)) (justify left))
-    )
-    (property "Footprint" "TerminalBlock_Phoenix:TerminalBlock_Phoenix_MKDS-1,5-2_1x02_P5.00mm_Horizontal" (id 2) (at 168.91 119.38 0)
-      (effects (font (size 1.27 1.27)) hide)
-    )
-    (property "Datasheet" "~" (id 3) (at 168.91 119.38 0)
-      (effects (font (size 1.27 1.27)) hide)
-    )
-    (pin "1")
-    (pin "2")
-  )
   (symbol (lib_id "power:GND") (at 163.83 59.69 270) (unit 1)
     (in_bom yes) (on_board yes) (fields_autoplaced)
@@
     )
     (pin "1")
-  )
-  (symbol (lib_id "Connector:Screw_Terminal_01x02") (at 168.91 133.35 0) (unit 1)
-    (in_bom yes) (on_board yes) (fields_autoplaced)
-    (property "Reference" "J10" (id 0) (at 171.45 133.3499 0)
-      (effects (font (size 1.27 1.27)) (justify left))
-    )
-    (property "Value" "MOTOR_D_OUT" (id 1) (at 171.45 135.8899 0)
-      (effects (font (size 1.27 1.27)) (justify left))
-    )
-    (property "Footprint" "TerminalBlock_Phoenix:TerminalBlock_Phoenix_MKDS-1,5-2_1x02_P5.00mm_Horizontal" (id 2) (at 168.91 133.35 0)
-      (effects (font (size 1.27 1.27)) hide)
-    )
-    (property "Datasheet" "~" (id 3) (at 168.91 133.35 0)
-      (effects (font (size 1.27 1.27)) hide)
-    )
-    (pin "1")
-    (pin "2")
   )
   (symbol (lib_id "Connector:Screw_Terminal_01x03") (at 168.91 62.23 0) (unit 1)
@@
     (pin "1")
   )
-  (symbol (lib_id "Connector:Conn_01x05_Female") (at 158.75 151.13 180) (unit 1)
-    (in_bom yes) (on_board yes) (fields_autoplaced)
-    (property "Reference" "J11" (id 0) (at 159.385 140.97 0))
-    (property "Value" "STEPPER_TERMINAL" (id 1) (at 159.385 143.51 0))
-    (property "Footprint" "Connector_PinHeader_2.54mm:PinHeader_1x05_P2.54mm_Vertical" (id 2) (at 158.75 151.13 0)
-      (effects (font (size 1.27 1.27)) hide)
-    )
-    (property "Datasheet" "~" (id 3) (at 158.75 151.13 0)
-      (effects (font (size 1.27 1.27)) hide)
-    )
+  (symbol (lib_id "Connector:Conn_01x05_Female") (at 158.75 123.19 180) (unit 1)
+    (in_bom yes) (on_board yes)
+    (property "Reference" "J11" (id 0) (at 167.64 113.03 0))
+    (property "Value" "STEPPER_TERMINAL" (id 1) (at 167.64 115.57 0))
+    (property "Footprint" "Connector_PinHeader_2.54mm:PinHeader_1x05_P2.54mm_Vertical" (id 2) (at 158.75 123.19 0)
+      (effects (font (size 1.27 1.27)) hide)
+    )
+    (property "Datasheet" "~" (id 3) (at 158.75 123.19 0)
+      (effects (font (size 1.27 1.27)) hide)
+    )
