File: ses-motor-shield/schematics/motor-schematic/dc_driver_ics.kicad_sch (KiCad schematic)
At the start: 3 parts, among them U2 L293D, U3 L293D, U5 L293D

Commit message: finished board
Other:
- note added: "*a total of 2 DC motors can be controlled by 2 ICs *a total of 1 stepper motors can be controlled by these 2 ICs"
- note removed: "*Add a stepper motor power toggle here"
- note removed: "*a total of 4 DC motors can be controlled by these 2 ICs *a total of 2 stepper motors can be controlled by these 2 ICs"
Changed lines of the file:
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@@
     (stroke (width 0) (type default) (color 0 0 0 0))
   )
-  (text "*a total of 4 DC motors can be controlled by these 2 ICs\n*a total of 2 stepper motors can be controlled by these 2 ICs\n"
+  (text "*a total of 2 DC motors can be controlled by 2 ICs\n*a total of 1 stepper motors can be controlled by these 2 ICs\n"
     (at 220.98 128.27 0)
     (effects (font (size 1.27 1.27)) (justify left bottom))
   )
-  (text "*Add a stepper motor power toggle here\n" (at 190.5 67.31 0)
-    (effects (font (size 1.27 1.27)) (justify left bottom))
-  )
