File: ses-motor-shield/schematics/motor-schematic/motor-schematic.kicad_pcb (KiCad board)
At the start: 2 copper layers, 71.1 x 69.1 mm, 34 parts, among them J1 EXTERNAL_MOTOR_POWER, J10 MOTOR_D_OUT, J11 STEPPER_TERMINAL, J2 Conn_01x03_Female, J3 Conn_01x20_Female, J4 Conn_01x20_Female, J5 SERVO1, J6 SERVO2, J7 MOTOR_A_OUT, J8 MOTOR_B_OUT, J9 MOTOR_C_OUT, Q1 Q_NMOS_DGS, Q2 TIP3055, U1 LM317_SOT-223, U2 L293D, U3 L293D, U4 AMS1117-5.0, U5 L293D, U6 AMS1117-3.3

Commit message: finished board
Parts:
- removed J10: MOTOR_D_OUT, TerminalBlock_Phoenix:TerminalBlock_Phoenix_MKDS-1,5-2_1x02_P5.00mm_Horizontal
- removed J9: MOTOR_C_OUT, TerminalBlock_Phoenix:TerminalBlock_Phoenix_MKDS-1,5-2_1x02_P5.00mm_Horizontal
- removed Q1: Q_NMOS_DGS, Package_TO_SOT_THT:TO-220-3_Vertical
- added D2: 1N4007, Diode_THT:D_DO-41_SOD81_P10.16mm_Horizontal, F.Cu at (63.2, 85.5)
- moved J7 6.58 mm to (66.5, 107.0), turned to 90 degrees
- moved J8 6.43 mm to (66.7, 119.8), turned to 90 degrees
- moved J1 4.40 mm to (65.7, 70.8), turned to 90 degrees
Connections:
- J1 pad 2: Net-(C6-Pad1) -> Net-(J1-Pad2)
- J11 pad 3: OUT3 -> OUT2
- J11 pad 4: OUT2 -> OUT3
Routing:
- net MOTOR_C_OUT+: track 56.7 -> 0.00 mm
- net MOTOR_C_OUT-: track 43.7 -> 0.00 mm
- net MOTOR_D_OUT+: track 40.7 -> 0.00 mm, vias 1 -> 0
- net SERVO_5V: track 87.4 -> 127.6 mm
- net MOTOR_D_OUT-: track 30.0 -> 0.00 mm, vias 1 -> 0
- net OUT3: track 44.5 -> 73.8 mm
- net GND: track 211.8 -> 183.2 mm
- net Net-(J1-Pad2): track 0.00 -> 23.7 mm
- net 12V: track 154.9 -> 136.2 mm, vias 0 -> 1
- net Net-(C6-Pad1): track 32.0 -> 45.3 mm, vias 0 -> 3
- net OUT2: track 66.6 -> 53.5 mm
- net MOTOR_A_OUT+: track 32.7 -> 44.4 mm
- net MOTOR_B_OUT-: track 76.2 -> 67.9 mm
- net MOTOR_B_OUT+: track 57.4 -> 62.6 mm
- net Net-(J2-Pad2): track 53.7 -> 54.9 mm
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- added copper zone on B.Cu, net GND
- added copper zone on F.Cu, net GND
Other:
- board text added: "-"
- board text removed: "MOTOR3"
- board text removed: "MOTOR4"
